File: Finger Print Scanner.brd (EAGLE design)
At the start: 99.7 x 99.7 mm, 63 parts, among them CN2 BATT_IN_JST, Q1 32.768kHz, U1 DS1307, U3 MCP73833T-AMI/MF, U4 PAM2401, U6 FT232RLSSOP

Commit message: Add files via upload
Parts:
- added R14: 1K, SparkFun:0805
Connections:
- removed net +5V: U6.20
- net 5V: now also U6.20
- net GND: now also R14.2
- net RESET: now also R14.1
Routing:
- net 5V: track 450.3 -> 463.1 mm, vias 10 -> 11
- net PC0: track 56.9 -> 63.4 mm
- net GND: track 168.1 -> 173.9 mm
- net RESET: track 48.6 -> 51.5 mm
Other:
- outline, holes or cut-outs redrawn
- board text removed: "Aaron Weiss, Patrick Alberts, Toni Klopfenstein"
- board text removed: "C:/Users/Derek/Pictures/Capture.bmp"
- board text removed: "Marshall Taylor"
- board text removed: "Open Source Hardware"
