File: Finger Print Scanner.sch (EAGLE design)
At the start: 63 parts, among them CN2 BATT_IN_JST, Q1 32.768kHz, U1 DS1307, U3 MCP73833T-AMI/MF, U4 PAM2401, U6 FT232RLSSOP, Y2 RESONATORMU

Commit message: Add files via upload
Parts:
- added R14: 1K, SparkFun:RESISTOR0805-RES
Connections:
- removed net +5V: U6.VCC
- net 5V: now also U6.VCC
- net GND: now also R14.2
- net RESET: now also R14.1
Other:
- moved on the sheet: C7
Changed lines of the file:
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@@
 <?xml version="1.0" encoding="utf-8"?>
 <!DOCTYPE eagle SYSTEM "eagle.dtd">
-<eagle version="8.7.1">
+<eagle version="9.0.0">
 <drawing>
 <settings>
@@
 <part name="J5" library="SparkFun-Connectors" deviceset="CONN_02" device=""/>
 <part name="SUPPLY6" library="SparkFun-Aesthetics" deviceset="5V" device=""/>
+<part name="R14" library="SparkFun" deviceset="RESISTOR" device="0805-RES" value="1K"/>
+<part name="GND13" library="supply1" deviceset="GND" device=""/>
 </parts>
 <sheets>
@@
 <instance part="RT10" gate="G$1" x="200.66" y="309.88" rot="R180"/>
 <instance part="GND4" gate="1" x="187.96" y="320.04" rot="R270"/>
-<instance part="C7" gate="G$1" x="-10.16" y="416.56" rot="R90"/>
+<instance part="C7" gate="G$1" x="-7.62" y="416.56" rot="R90"/>
 <instance part="C9" gate="G$1" x="-104.14" y="411.48"/>
 <instance part="GND12" gate="1" x="-104.14" y="403.86"/>
@@
 <attribute name="VALUE" x="-111.125" y="284.48" size="1.778" layer="96"/>
 </instance>
-<instance part="P+3" gate="1" x="-96.52" y="424.18" smashed="yes">
-<attribute name="VALUE" x="-94.615" y="426.72" size="1.778" layer="96" rot="R180"/>
+<instance part="P+3" gate="1" x="-99.06" y="424.18" smashed="yes">
+<attribute name="VALUE" x="-97.155" y="426.72" size="1.778" layer="96" rot="R180"/>
 </instance>
 <instance part="RT11" gate="G$1" x="68.58" y="363.22" smashed="yes" rot="R180">
@@
 <instance part="R13" gate="G$1" x="-2.54" y="353.06" rot="R90"/>
 <instance part="GND6" gate="1" x="2.54" y="347.98" rot="R90"/>
+<instance part="R14" gate="G$1" x="-17.78" y="421.64" rot="R90"/>
+<instance part="GND13" gate="1" x="-17.78" y="431.8" rot="R180"/>
 </instances>
 <busses>
@@
 <pinref part="GND6" gate="1" pin="GND"/>
 <wire x1="-2.54" y1="347.98" x2="0" y2="347.98" width="0.1524" layer="91"/>
+</segment>
+<segment>
+<pinref part="GND13" gate="1" pin="GND"/>
+<pinref part="R14" gate="G$1" pin="2"/>
+<wire x1="-17.78" y1="429.26" x2="-17.78" y2="426.72" width="0.1524" layer="91"/>
 </segment>
 </net>
@@
 <pinref part="SUPPLY21" gate="G$1" pin="5V"/>
 <wire x1="139.7" y1="332.74" x2="139.7" y2="335.28" width="0.1524" layer="91"/>
+</segment>
+<segment>
+<wire x1="-99.06" y1="421.64" x2="-81.28" y2="421.64" width="0.1524" layer="91"/>
+<pinref part="U6" gate="G$1" pin="VCC"/>
+<label x="-91.44" y="421.64" size="1.778" layer="95"/>
+<pinref part="P+3" gate="1" pin="+5V"/>
 </segment>
 </net>
@@
 </segment>
 </net>
-<net name="+5V" class="3">
-<segment>
-<wire x1="-96.52" y1="421.64" x2="-81.28" y2="421.64" width="0.1524" layer="91"/>
-<pinref part="U6" gate="G$1" pin="VCC"/>
-<label x="-91.44" y="421.64" size="1.778" layer="95"/>
-<pinref part="P+3" gate="1" pin="+5V"/>
-</segment>
-</net>
 <net name="AREF" class="4">
 <segment>
@@
 <junction x="0" y="421.64"/>
 <junction x="0" y="416.56"/>
-<wire x1="-7.62" y1="416.56" x2="0" y2="416.56" width="0.1524" layer="91"/>
+<wire x1="-5.08" y1="416.56" x2="0" y2="416.56" width="0.1524" layer="91"/>
 <pinref part="C7" gate="G$1" pin="2"/>
 <pinref part="ICSP" gate="A" pin="5"/>
@@
 <pinref part="U6" gate="G$1" pin="DTR"/>
 <pinref part="C7" gate="G$1" pin="1"/>
-<wire x1="-15.24" y1="416.56" x2="-50.8" y2="416.56" width="0.1524" layer="91"/>
-</segment>
-</net>
+<wire x1="-12.7" y1="416.56" x2="-17.78" y2="416.56" width="0.1524" layer="91"/>
+<pinref part="R14" gate="G$1" pin="1"/>
+<wire x1="-17.78" y1="416.56" x2="-50.8" y2="416.56" width="0.1524" layer="91"/>
+<junction x="-17.78" y="416.56"/>
+</segment>
+</net>
